File: Hardware/PCB Designs/1. PDU/atmgea_BISTandTelem.kicad_sch (KiCad schematic)
At the start: 16 parts, among them J7 Conn_01x08_Pin, SW1 SW_Push, U14 MAX481E, U6 ATmega8-16A, Y1 Crystal

Commit message: Update docs/index.md with new assets
Parts:
- added H5: MountingHole_Pad, MountingHole:MountingHole_3.2mm_M3_ISO7380_Pad, symbol Mechanical:MountingHole_Pad
Connections:
- net GND: now also H5.1
